File: pcb/p2000t-joystick-nes/p2000t-joystick-nes.kicad_sch (KiCad schematic)
At the start: 40 parts, among them J3 P2000T Port 2, SW1 KEYMAPPING, U1 74HC02, U2 74HC74, U3 74HC138, U4 74LS193, U5 74LS08, U6 SST39SF010, U7 SST39SF010, U8 74LS595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

Commit message: Pre-routing commit
Parts:
- removed C1, C2, C3, C4, C6, C8, C9: .1uF, Capacitor_THT:C_Disc_D5.0mm_W2.5mm_P5.00mm, symbol Device:C
- added U10: 74HC04, Package_DIP:DIP-14_W7.62mm_Socket, symbol 74xx:74HC04
- renumbered C5 to C1, C7 to C2
Connections:
- net CLK: now also U10.10, U10.13; no longer J1.2 (CLK), J2.2 (CLK), U4.5 (UP), U5.10, X1.8 (OUT)
- net GND: now also U10.7 (GND)
- net VCC: now also U10.14 (VCC)
- net at U5.6: now also U5.10; no longer U5.9
- net 500KHz: now reaches U4.3 (QA), U5.1
- net 500KHz: now also U10.1
- net at U5.3: now also U5.9; no longer U5.4
- net at U4.6 (QC): now also U5.4; no longer U5.5
- net at U4.7 (QD): now also U5.5
- new net: U10.2, U10.3
- new net: U10.4, U10.5
- new net: U4.5 (UP), X1.8 (OUT)
- new net: U10.6, U10.9
- new net: U10.11, U10.8
- new net CTRLCLK: J1.2 (CLK), J2.2 (CLK), U10.12
- no-connect marks 26 -> 29
Other:
- note added: "Controller CLK signal is slightly delayed with respect to LATCH"
- note added: "Shift register reads half a cycle after controller clock"
- moved on the sheet: U4, U5A, U5B, U5C, U5D, U5E, X1

Commit message: Routing
Parts:
- U4: value 74LS193 -> 74HC193
- U5: value 74LS08 -> 74HC08
- U8, U9: value 74LS595 -> 74HC595
Changed lines of the file:
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@@
 			)
 		)
-		(property "Value" "74LS08"
+		(property "Value" "74HC08"
 			(at 106.6717 210.82 0)
 			(effects
@@
 			)
 		)
-		(property "Value" "74LS08"
+		(property "Value" "74HC08"
 			(at 118.1017 184.15 0)
 			(effects
@@
 			)
 		)
-		(property "Value" "74LS08"
+		(property "Value" "74HC08"
 			(at 100.3217 171.45 0)
 			(effects
@@
 			)
 		)
-		(property "Value" "74LS08"
+		(property "Value" "74HC08"
 			(at 100.3217 186.69 0)
 			(effects
@@
 			)
 		)
-		(property "Value" "74LS595"
+		(property "Value" "74HC595"
 			(at 234.6041 200.66 0)
 			(effects
@@
 			)
 		)
-		(property "Value" "74LS08"
+		(property "Value" "74HC08"
 			(at 133.35 209.55 90)
 			(effects
@@
 			)
 		)
-		(property "Value" "74LS193"
+		(property "Value" "74HC193"
 			(at 70.7741 177.8 0)
 			(effects
@@
 			)
 		)
-		(property "Value" "74LS595"
+		(property "Value" "74HC595"
 			(at 234.6041 149.86 0)
 			(effects
