File: pcb/p2000t-joystick-slot2-cpld/p2000t-joystick-slot2-cpld.kicad_pcb (KiCad board)
At the start: 2 copper layers, 80 x 100 mm, 24 parts, among them J1 PLAYER1, J2 P2000T Port 2, J3 PLAYER2, J4 Atmel-JTAG-10, J5 POWER, SW1 SW_DIP_x02, U3 ATF1502ASV

Commit message: Fixing design and CUPL
Parts:
- U3: value ATF1502ASV -> ATF1502AS
Connections:
- U3 pad 16: unconnected-(U3-I/O-Pad16) -> D6
Routing:
- net D6: track 23.9 -> 61.0 mm, vias 0 -> 5
- net Net-(D8-K): track 14.0 -> 19.6 mm
Other:
- board text added: "/rev1/"
- board text added: "CPLD VERSION"
- board text added: "PHILIPS P2000T JOYSTICK CARTRIDGE"
- board text added: "VCC"
- board text added: "connect to program using ATDH1150USB"
